Commit message: Remove in favor of a combined robot package

File: model/conveyor_belt/conveyor.urdf (robot description, URDF)
Before this commit: robot conveyor_belt, 10 links, 9 joints
Links:
- removed link world
Joints:
- removed joint joint_belt

Commit message: Switch mesh uri's to what rviz expects.
This breaks this package for Gazebo

File: model/conveyor_belt/conveyor.urdf (robot description, URDF)
Before this commit: robot conveyor_belt, 9 links, 8 joints
Links:
- link link_belt: geometry visual mesh filename=package://conveyor_belt/model/conveyor_belt/meshes/belt.dae scale=0.001 0.001 0.001
- link link_bridge_left: geometry visual mesh filename=package://conveyor_belt/model/conveyor_belt/meshes/bridge_l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 scale=0.001 0.001 0.001
- link link_bridge_right: geometry visual mesh filename=package://conveyor_belt/model/conveyor_belt/meshes/bridge_r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 scale=0.001 0.001 0.001
- link link_flap_back: geometry visual mesh filename=package://conveyor_belt/model/conveyor_belt/meshes/flap_bac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 scale=0.001 0.001 0.001
- link link_flap_front: geometry visual mesh filename=package://conveyor_belt/model/conveyor_belt/meshes/flap_fro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 scale=0.001 0.001 0.001
- link link_leg_back_left: geometry visual mesh filename=package://conveyor_belt/model/conveyor_belt/meshes/leg_back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 scale=0.001 0.001 0.001
- link link_leg_back_right: geometry visual mesh filename=package://conveyor_belt/model/conveyor_belt/meshes/leg_back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 scale=0.001 0.001 0.001
- link link_leg_front_left: geometry visual mesh filename=package://conveyor_belt/model/conveyor_belt/meshes/leg_fron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 scale=0.001 0.001 0.001
- link link_leg_front_right: geometry visual mesh filename=package://conveyor_belt/model/conveyor_belt/meshes/leg_fron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 scale=0.001 0.001 0.001

Commit message: New conveyor belt model

File: model/conveyor_belt/conveyor.urdf (robot description, URDF)
Before this commit: robot conveyor_belt, 9 links, 8 joints
Links:
- added link conveyor_base, mass 0.001
- link link_belt: mass 0.001 -> 10.0; geometry collision box size=6.10862 0.67785 0.01; visual mesh filename=package://conveyor_belt/model/conveyor_belt/meshes/belt.dae scale=1.0 1.0 1.0
- link link_bridge_left: mass 0.001 -> 10.0; geometry collision box size=0.0254 0.67785 0.127; visual mesh filename=package://conveyor_belt/model/conveyor_belt/meshes/bridge_l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 scale=1.0 1.0 1.0
- link link_bridge_right: mass 0.001 -> 10.0; geometry collision box size=0.0254 0.67785 0.127; visual mesh filename=package://conveyor_belt/model/conveyor_belt/meshes/brigde_r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 scale=1.0 1.0 1.0
- link link_flap_back: mass 0.001 -> 10.0; geometry collision box size=6.10862 0.02857 0.07937; visual mesh filename=package://conveyor_belt/model/conveyor_belt/meshes/flap_bac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 scale=1.0 1.0 1.0
- link link_flap_front: mass 0.001 -> 10.0; geometry collision box size=6.10862 0.02857 0.07937; visual mesh filename=package://conveyor_belt/model/conveyor_belt/meshes/flap_fro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 scale=1.0 1.0 1.0
- link link_leg_back_left: mass 0.001 -> 10.0; geometry collision box size=0.0508 0.0508 1.24458; visual mesh filename=package://conveyor_belt/model/conveyor_belt/meshes/leg_back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 scale=1.0 1.0 1.0
- link link_leg_back_right: mass 0.001 -> 10.0; geometry collision box size=0.0508 0.0508 1.24458; visual mesh filename=package://conveyor_belt/model/conveyor_belt/meshes/leg_back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 scale=1.0 1.0 1.0
- link link_leg_front_left: mass 0.001 -> 10.0; geometry collision box size=0.0508 0.0508 1.24458; visual mesh filename=package://conveyor_belt/model/conveyor_belt/meshes/leg_fron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 scale=1.0 1.0 1.0
- link link_leg_front_right: mass 0.001 -> 10.0; geometry collision box size=0.0508 0.0508 1.24458; visual mesh filename=package://conveyor_belt/model/conveyor_belt/meshes/leg_fron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 scale=1.0 1.0 1.0
Joints:
- added joint joint_belt: type fixed, parent conveyor_base, child link_belt, origin xyz=0 0.33893 -0.08438 rpy=0 0 0
- joint joint_bridge_left: origin xyz=0.59689 0.3048 1.23014 rpy=0 0 0 -> xyz=0.62864 0.33893 0.05714 rpy=0 0 0; parent world -> conveyor_base
- joint joint_bridge_right: origin xyz=-0.85089 0.3048 1.23014 rpy=0 0 0 -> xyz=-1.79703 0.33893 0.05714 rpy=0 0 0; parent world -> conveyor_base
- joint joint_flap_back: origin xyz=0 0.0127 1.182 rpy=0 0 0 -> xyz=0 0.01429 -0.03969 rpy=0 0 0; parent world -> conveyor_base
- joint joint_flap_front: origin xyz=0 0.59689 1.182 rpy=0 0 0 -> xyz=0 0.66357 -0.03969 rpy=0 0 0; parent world -> conveyor_base
- joint joint_leg_back_left: origin xyz=0.68579 -0.0254 0.556 rpy=0 0 0 -> xyz=1.68273 -0.0254 -0.6223 rpy=0 0 0; parent world -> conveyor_base
- joint joint_leg_back_right: origin xyz=-0.68579 -0.0254 0.556 rpy=0 0 0 -> xyz=-1.68273 -0.0254 -0.6223 rpy=0 0 0; parent world -> conveyor_base
- joint joint_leg_front_left: origin xyz=0.68579 0.63499 0.556 rpy=0 0 0 -> xyz=1.68273 0.70325 -0.6223 rpy=0 0 0; parent world -> conveyor_base
- joint joint_leg_front_right: origin xyz=-0.68579 0.63499 0.556 rpy=0 0 0 -> xyz=-1.68273 0.70325 -0.6223 rpy=0 0 0; parent world -> conveyor_base
